Commit message: Prep for revisit

File: traxster_description/urdf/traxster.urdf (robot description, URDF)
Before this commit: robot traxster, 16 links, 15 joints
Links:
- link camera_link: geometry collision box size=0.0730 .2760 0.0720; visual mesh filename=package://traxster_description/meshes/vggvct.dae scale=73 73 73
